File: AU_MacroPad.sch (EAGLE design)
At the start: 95 parts, among them IC1 74HCT1G125DBV, IC3 RP2040_QFN56, SW2 RA SW, SW3 EN11-VSM1AF15, U1 W25Q64, U2 RT9080-3.3, U3 PAM8302, X1 TYPE C, X2 ZJY130-2864KSWLG22, Y1 12MHz/12pF

Commit message: swap gnd and usbboot to match original macropad
Connections:
- net GND: now also SW3.D; no longer SW3.E
- net USBBOOT: now also SW3.E; no longer SW3.D
Changed lines of the file:
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@@
 <attribute name="VALUE" x="147.32" y="137.16" size="1.778" layer="96"/>
 </instance>
-<instance part="GND43" gate="1" x="134.62" y="139.7" smashed="yes" rot="MR0">
-<attribute name="VALUE" x="137.16" y="137.16" size="1.778" layer="96" rot="MR0"/>
+<instance part="GND43" gate="1" x="134.62" y="152.4" smashed="yes" rot="MR180">
+<attribute name="VALUE" x="132.08" y="154.94" size="1.778" layer="96" rot="MR180"/>
 </instance>
 <instance part="GND44" gate="1" x="172.72" y="137.16" smashed="yes" rot="MR0">
@@
 </segment>
 <segment>
-<wire x1="137.16" y1="144.78" x2="134.62" y2="144.78" width="0.1524" layer="91"/>
-<wire x1="134.62" y1="144.78" x2="134.62" y2="142.24" width="0.1524" layer="91"/>
+<wire x1="137.16" y1="149.86" x2="134.62" y2="149.86" width="0.1524" layer="91"/>
 <pinref part="GND43" gate="1" pin="GND"/>
-<pinref part="SW3" gate="G$1" pin="E"/>
+<pinref part="SW3" gate="G$1" pin="D"/>
 </segment>
 <segment>
@@
 <pinref part="C15" gate="G$1" pin="2"/>
 <pinref part="X2" gate="G$1" pin="C1+"/>
-</segment>
-</net>
-<net name="USBBOOT" class="0">
-<segment>
-<wire x1="137.16" y1="149.86" x2="127" y2="149.86" width="0.1524" layer="91"/>
-<label x="127" y="149.86" size="1.778" layer="95"/>
-<pinref part="SW3" gate="G$1" pin="D"/>
 </segment>
 </net>
@@
 </segment>
 </net>
+<net name="USBBOOT" class="0">
+<segment>
+<pinref part="SW3" gate="G$1" pin="E"/>
+<wire x1="137.16" y1="144.78" x2="127" y2="144.78" width="0.1524" layer="91"/>
+<label x="127" y="144.78" size="1.778" layer="95"/>
+</segment>
+</net>

Commit message: add bottom fiducials, clean up silk due to other side OLED
Parts:
- added U$79, U$83: FIDUCIAL_1MM, microbuilder:FIDUCIAL_1MM
- X2: value ZJY130-2864KSWLG22 -> ZJY130-2864KSWLG22_CONN; device adafruit_display:ZJY130-2864KSWLG22 -> adafruit_display:ZJY130-2864KSWLG22_CONN
Changed lines of the file:
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@@
 <grid distance="0.1" unitdist="inch" unit="inch" style="lines" multiple="1" display="no" altdistance="0.01" altunitdist="inch" altunit="inch"/>
 <layers>
-<layer number="1" name="Top" color="4" fill="1" visible="no" active="no"/>
-<layer number="2" name="Route2" color="16" fill="3" visible="no" active="no"/>
-<layer number="3" name="Route3" color="17" fill="3" visible="no" active="no"/>
-<layer number="4" name="Route4" color="18" fill="4" visible="no" active="no"/>
-<layer number="5" name="Route5" color="19" fill="4" visible="no" active="no"/>
-<layer number="6" name="Route6" color="25" fill="8" visible="no" active="no"/>
-<layer number="7" name="Route7" color="26" fill="8" visible="no" active="no"/>
-<layer number="8" name="Route8" color="27" fill="2" visible="no" active="no"/>
-<layer number="9" name="Route9" color="28" fill="2" visible="no" active="no"/>
-<layer number="10" name="Route10" color="29" fill="7" visible="no" active="no"/>
-<layer number="11" name="Route11" color="30" fill="7" visible="no" active="no"/>
-<layer number="12" name="Route12" color="20" fill="5" visible="no" active="no"/>
-<layer number="13" name="Route13" color="21" fill="5" visible="no" active="no"/>
-<layer number="14" name="Route14" color="22" fill="6" visible="no" active="no"/>
-<layer number="15" name="Route15" color="23" fill="6" visible="no" active="no"/>
-<layer number="16" name="Bottom" color="1" fill="1" visible="no" active="no"/>
-<layer number="17" name="Pads" color="2" fill="1" visible="no" active="no"/>
-<layer number="18" name="Vias" color="2" fill="1" visible="no" active="no"/>
-<layer number="19" name="Unrouted" color="6" fill="1" visible="no" active="no"/>
-<layer number="20" name="Dimension" color="24" fill="1" visible="no" active="no"/>
-<layer number="21" name="tPlace" color="7" fill="1" visible="no" active="no"/>
-<layer number="22" name="bPlace" color="7" fill="1" visible="no" active="no"/>
-<layer number="23" name="tOrigins" color="15" fill="1" visible="no" active="no"/>
-<layer number="24" name="bOrigins" color="15" fill="1" visible="no" active="no"/>
-<layer number="25" name="tNames" color="7" fill="1" visible="no" active="no"/>
-<layer number="26" name="bNames" color="7" fill="1" visible="no" active="no"/>
-<layer number="27" name="tValues" color="7" fill="1" visible="no" active="no"/>
-<layer number="28" name="bValues" color="7" fill="1" visible="no" active="no"/>
+<layer number="1" name="Top" color="4" fill="1" visible="yes" active="no"/>
+<layer number="2" name="Route2" color="16" fill="3" visible="yes" active="no"/>
+<layer number="3" name="Route3" color="17" fill="3" visible="yes" active="no"/>
+<layer number="4" name="Route4" color="18" fill="4" visible="yes" active="no"/>
+<layer number="5" name="Route5" color="19" fill="4" visible="yes" active="no"/>
+<layer number="6" name="Route6" color="25" fill="8" visible="yes" active="no"/>
+<layer number="7" name="Route7" color="26" fill="8" visible="yes" active="no"/>
+<layer number="8" name="Route8" color="27" fill="2" visible="yes" active="no"/>
+<layer number="9" name="Route9" color="28" fill="2" visible="yes" active="no"/>
+<layer number="10" name="Route10" color="29" fill="7" visible="yes" active="no"/>
+<layer number="11" name="Route11" color="30" fill="7" visible="yes" active="no"/>
+<layer number="12" name="Route12" color="20" fill="5" visible="yes" active="no"/>
+<layer number="13" name="Route13" color="21" fill="5" visible="yes" active="no"/>
+<layer number="14" name="Route14" color="22" fill="6" visible="yes" active="no"/>
+<layer number="15" name="Route15" color="23" fill="6" visible="yes" active="no"/>
+<layer number="16" name="Bottom" color="1" fill="1" visible="yes" active="no"/>
+<layer number="17" name="Pads" color="2" fill="1" visible="yes" active="no"/>
+<layer number="18" name="Vias" color="2" fill="1" visible="yes" active="no"/>
+<layer number="19" name="Unrouted" color="6" fill="1" visible="yes" active="no"/>
+<layer number="20" name="Dimension" color="24" fill="1" visible="yes" active="no"/>
+<layer number="21" name="tPlace" color="7" fill="1" visible="yes" active="no"/>
+<layer number="22" name="bPlace" color="7" fill="1" visible="yes" active="no"/>
+<layer number="23" name="tOrigins" color="15" fill="1" visible="yes" active="no"/>
+<layer number="24" name="bOrigins" color="15" fill="1" visible="yes" active="no"/>
+<layer number="25" name="tNames" color="7" fill="1" visible="yes" active="no"/>
+<layer number="26" name="bNames" color="7" fill="1" visible="yes" active="no"/>
+<layer number="27" name="tValues" color="7" fill="1" visible="yes" active="no"/>
+<layer number="28" name="bValues" color="7" fill="1" visible="yes" active="no"/>
 <layer number="29" name="tStop" color="7" fill="3" visible="no" active="no"/>
 <layer number="30" name="bStop" color="7" fill="6" visible="no" active="no"/>
@@
 <layer number="35" name="tGlue" color="7" fill="4" visible="no" active="no"/>
 <layer number="36" name="bGlue" color="7" fill="5" visible="no" active="no"/>
-<layer number="37" name="tTest" color="7" fill="1" visible="no" active="no"/>
-<layer number="38" name="bTest" color="7" fill="1" visible="no" active="no"/>
+<layer number="37" name="tTest" color="7" fill="1" visible="yes" active="no"/>
+<layer number="38" name="bTest" color="7" fill="1" visible="yes" active="no"/>
 <layer number="39" name="tKeepout" color="4" fill="11" visible="no" active="no"/>
 <layer number="40" name="bKeepout" color="1" fill="11" visible="no" active="no"/>
@@
 <layer number="44" name="Drills" color="7" fill="1" visible="no" active="no"/>
 <layer number="45" name="Holes" color="7" fill="1" visible="no" active="no"/>
-<layer number="46" name="Milling" color="3" fill="1" visible="no" active="no"/>
-<layer number="47" name="Measures" color="7" fill="1" visible="no" active="no"/>
-<layer number="48" name="Document" color="7" fill="1" visible="no" active="no"/>
-<layer number="49" name="Reference" color="7" fill="1" visible="no" active="no"/>
-<layer number="50" name="dxf" color="7" fill="1" visible="no" active="no"/>
-<layer number="51" name="tDocu" color="7" fill="1" visible="no" active="no"/>
-<layer number="52" name="bDocu" color="7" fill="1" visible="no" active="no"/>
-<layer number="53" name="tGND_GNDA" color="7" fill="9" visible="no" active="no"/>
-<layer number="54" name="bGND_GNDA" color="7" fill="9" visible="no" active="no"/>
-<layer number="56" name="wert" color="7" fill="1" visible="no" active="no"/>
-<layer number="57" name="tCAD" color="7" fill="1" visible="no" active="no"/>
-<layer number="58" name="b3D" color="7" fill="1" visible="no" active="no"/>
-<layer number="59" name="tCarbon" color="7" fill="1" visible="no" active="no"/>
-<layer number="60" name="bCarbon" color="7" fill="1" visible="no" active="no"/>
-<layer number="61" name="stand" color="7" fill="1" visible="no" active="no"/>
+<layer number="46" name="Milling" color="3" fill="1" visible="yes" active="no"/>
+<layer number="47" name="Measures" color="7" fill="1" visible="yes" active="no"/>
+<layer number="48" name="Document" color="7" fill="1" visible="yes" active="no"/>
+<layer number="49" name="Reference" color="7" fill="1" visible="yes" active="no"/>
+<layer number="50" name="dxf" color="7" fill="1" visible="yes" active="no"/>
+<layer number="51" name="tDocu" color="7" fill="1" visible="yes" active="no"/>
+<layer number="52" name="bDocu" color="7" fill="1" visible="yes" active="no"/>
+<layer number="53" name="tGND_GNDA" color="7" fill="9" visible="yes" active="no"/>
+<layer number="54" name="bGND_GNDA" color="7" fill="9" visible="yes" active="no"/>
+<layer number="56" name="wert" color="7" fill="1" visible="yes" active="no"/>
+<layer number="57" name="tCAD" color="7" fill="1" visible="yes" active="no"/>
+<layer number="58" name="b3D" color="7" fill="1" visible="yes" active="no"/>
+<layer number="59" name="tCarbon" color="7" fill="1" visible="yes" active="no"/>
+<layer number="60" name="bCarbon" color="7" fill="1" visible="yes" active="no"/>
+<layer number="61" name="stand" color="7" fill="1" visible="yes" active="no"/>
 <layer number="88" name="SimResults" color="9" fill="1" visible="yes" active="yes"/>
 <layer number="89" name="SimProbes" color="9" fill="1" visible="yes" active="yes"/>
@@
 <part name="TP2" library="adafruit_electromech" deviceset="SEWTAP" device="_SMTNUTM3"/>
 <part name="TP4" library="adafruit_electromech" deviceset="SEWTAP" device="_SMTNUTM3"/>
-<part name="X2" library="adafruit_display" deviceset="ZJY130-2864KSWLG22" device=""/>
+<part name="X2" library="adafruit_display" deviceset="ZJY130-2864KSWLG22" device="_CONN" value="ZJY130-2864KSWLG22_CONN"/>
 <part name="U$59" library="microbuilder" deviceset="GND" device=""/>
 <part name="C14" library="microbuilder" deviceset="CAP_CERAMIC" device="0805-NOOUTLINE" value="10uF"/>
@@
 <part name="GND47" library="supply1" deviceset="GND" device=""/>
 <part name="GND55" library="supply1" deviceset="GND" device=""/>
+<part name="U$79" library="microbuilder" deviceset="FIDUCIAL" device="_1MM"/>
+<part name="U$83" library="microbuilder" deviceset="FIDUCIAL" device="_1MM"/>
 </parts>
 <sheets>
@@
 <attribute name="VALUE" x="149.86" y="60.96" size="1.778" layer="96"/>
 </instance>
+<instance part="U$79" gate="G$1" x="220.98" y="35.56" smashed="yes"/>
+<instance part="U$83" gate="G$1" x="226.06" y="35.56" smashed="yes"/>
 </instances>
 <busses>
